File: Whale_Gosth/KiCad/Whale_Gosth.sch (KiCad schematic (older format))
At the start: 13 parts

Commit message: pcb v1.0
Parts:
- removed Regu_5V1: Screw_Terminal_1x03, Connectors_Terminal_Blocks:TerminalBlock_bornier-3_P5.08mm, symbol Screw_Terminal_1x03
- added J1, J2, J3, J4: CONN_01X01, Wire_Pads:SolderWirePad_single_2mmDrill, symbol CONN_01X01
Connections:
- net +24V: now also J2.1 (P1)
- net GND: now also J3.1 (P1)
- net at ESP-G1.19 (P19): now also J4.1 (P1)
Changed lines of the file:
@@
 $EndDescr
 $Comp
-L +24V #PWR1
+L +24V #PWR01
 U 1 1 5A786DA5
 P 1700 750
-F 0 "#PWR1" H 1700 600 50  0001 C CNN
+F 0 "#PWR01" H 1700 600 50  0001 C CNN
 F 1 "+24V" H 1700 890 50  0000 C CNN
 F 2 "" H 1700 750 50  0001 C CNN
@@
 SVN
 $Comp
-L GND #PWR2
+L GND #PWR02
 U 1 1 5A78ED88
 P 1700 4850
-F 0 "#PWR2" H 1700 4600 50  0001 C CNN
+F 0 "#PWR02" H 1700 4600 50  0001 C CNN
 F 1 "GND" H 1700 4700 50  0000 C CNN
 F 2 "" H 1700 4850 50  0001 C CNN
@@
 Connection ~ 1700 2800
 Wire Wire Line
-	1250 3800 1600 3800
-Wire Wire Line
-	1600 3800 1600 2400
-Connection ~ 1600 2400
-Wire Wire Line
-	1250 4000 1700 4000
-Connection ~ 1700 4000
-Wire Wire Line
 	1500 3000 1250 3000
 Connection ~ 1700 4750
@@
 	6550 6450 6550 6100
 Wire Wire Line
-	1250 4200 2600 4200
-Wire Wire Line
-	2600 4200 2600 4150
-Wire Wire Line
-	2600 4150 2650 4150
-Wire Wire Line
 	4200 2350 5150 2350
 Wire Wire Line
@@
 Wire Wire Line
 	6750 6300 6750 6100
-$Comp
-L Screw_Terminal_1x03 Regu_5V1
-U 1 1 5A798B47
-P 1050 4000
-F 0 "Regu_5V1" H 1050 4350 50  0000 C TNN
-F 1 "Screw_Terminal_1x03" V 900 4000 50  0000 C TNN
-F 2 "Connectors_Terminal_Blocks:TerminalBlock_bornier-3_P5.08mm" H 1050 3675 50  0001 C CNN
-F 3 "" H 1025 4100 50  0001 C CNN
-	1    1050 4000
-	1    0    0    -1
-$EndComp
 $Comp
 L 1902547 OUT_24V1
@@
 	1200 1300 2200 1300
 Connection ~ 2000 1300
+$Comp
+L CONN_01X01 J1
+U 1 1 5A7A0F0C
+P 1050 3600
+F 0 "J1" H 1050 3700 50  0000 C CNN
+F 1 "CONN_01X01" V 1150 3600 50  0000 C CNN
+F 2 "Wire_Pads:SolderWirePad_single_2mmDrill" H 1050 3600 50  0001 C CNN
+F 3 "" H 1050 3600 50  0001 C CNN
+	1    1050 3600
+	-1   0    0    1
+$EndComp
+$Comp
+L CONN_01X01 J2
+U 1 1 5A7A0FD5
+P 1050 3800
+F 0 "J2" H 1050 3900 50  0000 C CNN
+F 1 "CONN_01X01" V 1150 3800 50  0000 C CNN
+F 2 "Wire_Pads:SolderWirePad_single_2mmDrill" H 1050 3800 50  0001 C CNN
+F 3 "" H 1050 3800 50  0001 C CNN
+	1    1050 3800
+	-1   0    0    1
+$EndComp
+$Comp
+L CONN_01X01 J3
+U 1 1 5A7A101A
+P 1050 4000
+F 0 "J3" H 1050 4100 50  0000 C CNN
+F 1 "CONN_01X01" V 1150 4000 50  0000 C CNN
+F 2 "Wire_Pads:SolderWirePad_single_2mmDrill" H 1050 4000 50  0001 C CNN
+F 3 "" H 1050 4000 50  0001 C CNN
+	1    1050 4000
+	-1   0    0    1
+$EndComp
+$Comp
+L CONN_01X01 J4
+U 1 1 5A7A1059
+P 1050 4200
+F 0 "J4" H 1050 4300 50  0000 C CNN
+F 1 "CONN_01X01" V 1150 4200 50  0000 C CNN
+F 2 "Wire_Pads:SolderWirePad_single_2mmDrill" H 1050 4200 50  0001 C CNN
+F 3 "" H 1050 4200 50  0001 C CNN
+	1    1050 4200
+	-1   0    0    1
+$EndComp
+Wire Wire Line
+	2650 4150 1350 4150
+Wire Wire Line
+	1350 4150 1350 4200
+Wire Wire Line
+	1350 4200 1250 4200
+Wire Wire Line
+	1250 4000 2000 4000
+Connection ~ 2000 4000
+Wire Wire Line
+	1250 3800 1450 3800
+Wire Wire Line
+	1450 3800 1450 2400
+Connection ~ 1450 2400
 $EndSCHEMATC

Commit message: v2
Parts:
- added Buck_converter2: BUCK-CONVERTER2, Connectors_Terminal_Blocks:TerminalBlock_bornier-4_P5.08mm, symbol Screw_Terminal_1x04
- added Buck_converter3: BUCK-CONVERTER3, Connectors_Terminal_Blocks:TerminalBlock_bornier-4_P5.08mm, symbol Screw_Terminal_1x04
- Buck_converter1: value BUCK-CONVERTER -> BUCK-CONVERTER1
Connections:
- net +24V: now also Buck_converter2.1, Buck_converter3.1
- net GND: now also Buck_converter2.2, Buck_converter2.3, Buck_converter3.2, Buck_converter3.3
- new net: Buck_converter1.4, WS_0.1, WS_1.1
- new net: Buck_converter2.4, WS_2.1, WS_3.1
- new net: Buck_converter3.4, WS_4.1, WS_5.1
Other:
- moved on the sheet: Buck_converter1
