File: Whale_Gosth/KiCad/_autosave-Whale_Gosth.kicad_pcb (KiCad board)
At the start: 2 copper layers, 150 x 50 mm, 18 parts

Commit message: v2
Parts:
- added ?: SolderWirePad_single_2-5mmDrill, Wire_Pads:SolderWirePad_single_2-5mmDrill, B.Cu at (92.0, 94.0)
- added ?: SolderWirePad_single_2-5mmDrill, Wire_Pads:SolderWirePad_single_2-5mmDrill, B.Cu at (224.0, 95.0)
- added ?: SolderWirePad_single_2-5mmDrill, Wire_Pads:SolderWirePad_single_2-5mmDrill, B.Cu at (101.0, 104.0)
- added ?: logo_pitaya, riri:logo_pitaya, F.Cu at (224.0, 81.0)
- added ?: SolderWirePad_single_2-5mmDrill, Wire_Pads:SolderWirePad_single_2-5mmDrill, B.Cu at (215.0, 104.0)
- added REF**: , Wire_Pads:SolderWirePad_single_2-5mmDrill, F.Cu at (93.0, 83.0)
Routing:
- net SD3: track 44.6 -> 72.5 mm
- net CMD: track 38.3 -> 63.7 mm
- net +24V: track 176.2 -> 189.8 mm, vias 2 -> 0
Other:
- board size 150 x 50 mm -> 150 x 51 mm
- net class Default: clearance 1 -> 0.5; trace_width 2 -> 1
- rule trace_clearance: 1 -> 0.5
- board text added: "+"
- board text added: "-"
- board text added: "24"
- board text added: "3v3"
- board text added: "5"
- board text added: "5v"
- board text added: "By Riri"
- board text added: "CLK"
- board text added: "CMD"
- board text added: "Data"
- board text added: "EN"
- board text added: "ESP 32 WROOM"
- board text added: "GND"
- board text added: "Gnd"
- board text added: "IO0"
- board text added: "IO12"
- board text added: "IO13"
- board text added: "IO14"
- board text added: "IO15"
- board text added: "IO16"
- board text added: "IO17"
- board text added: "IO2"
- board text added: "IO25"
- board text added: "IO26"
- board text added: "IO27"
- board text added: "IO32"
- board text added: "IO33"
- board text added: "IO34"
- board text added: "IO35"
- board text added: "RXD0"
- board text added: "Regu. 7 V"
- board text added: "SD0"
- board text added: "SD1"
- board text added: "SD2"
- board text added: "SD3"
- board text added: "SVN"
- board text added: "SVP"
- board text added: "TXD0"
- board text added: "Whale Gosth V 2.0"
- board text added: "clk"
- board text added: "gnd"
